File: pcb/coyote-pcb.kicad_pcb (KiCad board)
At the start: 2 copper layers, 106 x 47 mm, 17 parts, among them U1 Basalt

Commit message: Add silkscreen logo etc, update title blocks
Routing:
- net +5V: track 99.5 -> 98.5 mm
Other:
- board text added: "Coyote Rev${REVISION}"
- board text added: "github.com/oc-ece-mesa"
